File: Eagle/testscreen_4x4.brd (EAGLE design)
At the start: 160 x 100 mm, 33 parts, among them U1 WS2812, U10 WS2812, U11 WS2812, U12 WS2812, U13 WS2812, U14 WS2812, U15 WS2812, U16 WS2812, U2 WS2812, U3 WS2812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

Commit message: developing esp32 version on new branch
Other:
- board text added: "TOP"
Changed lines of the file:
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@@
 <wire x1="160" y1="100" x2="0" y2="100" width="0" layer="20"/>
 <wire x1="0" y1="100" x2="0" y2="0" width="0" layer="20"/>
+<text x="43.18" y="45.72" size="2.54" layer="51" font="vector" ratio="18">TOP</text>
 </plain>
 <attributes>
