File: Eagle/groovegrid_v2.brd (EAGLE design)
At the start: 160 x 100 mm, 33 parts, among them U1 WS2812, U10 WS2812, U11 WS2812, U12 WS2812, U13 WS2812, U14 WS2812, U15 WS2812, U16 WS2812, U2 WS2812, U3 WS2812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

Commit message: renamed to groovegrid v2
Parts:
- added B1: ESP32_DEVKITC_W_ANT_KEEPOUT, philmalessa:ESP32_DEVKITC
- added C17: 100n, resistor:C0805
- added R1, R2: 330, resistor:R0805
Connections:
- new net DATA_DEMO: R2.2, U1.2
- new net N$14: B1.P14, R1.1
- new net N$15: B1.P15, R2.1
- net +5V: now also B1.P20, C17.2
- net DATA: now also R1.2; no longer U1.2
- net GND: now also B1.P25, B1.P7, C17.1
