File: Eagle/groovegrid_v2.sch (EAGLE design)
At the start: 33 parts, among them U1 WS2812, U10 WS2812, U11 WS2812, U12 WS2812, U13 WS2812, U14 WS2812, U15 WS2812, U16 WS2812, U2 WS2812, U3 WS2812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

Commit message: renamed to groovegrid v2
Parts:
- added B1: ESP32_DEVKITC_W_ANT_KEEPOUT, philmalessa:ESP32_DEVKITC_W_ANT_KEEPOUT
- added C17: 100n, resistor:C-EUC0805
- added R1, R2: 330, resistor:R-EU_R0805
Connections:
- new net DATA_DEMO: R2.2, U1.DI
- new net N$14: B1.IO0, R1.1
- new net N$15: B1.IO2, R2.1
- net +5V: now also B1.5V, C17.2
- net DATA: now also R1.2; no longer U1.DI
- net GND: now also B1.GND, B1.GND@3, C17.1
Other:
- note removed: "CHECK PINOUT"
- moved on the sheet: X1-1, X1-2, X1-3
